Commit message: Atualização da navegação autonoma
Stack mais atualizado referente à navegação autonoma, com mudanças no urdf, parâmetros e etc

File: Computacional/robot/ros_ws/src/autonomous_drive/description/imu.xacro (robot description, xacro)
@@ -1,4 +1,5 @@
 <?xml version="1.0"?>
 <robot xmlns:xacro="http://www.ros.org/wiki/xacro">
+<!-- Esse arquivo descreve como o IMU foi tratado na simulação -->
     <xacro:property name="imu_x" value="0.15"/>
     <xacro:property name="imu_y" value="0.0"/>
@@ -9,5 +10,5 @@
     <xacro:property name="imu_topic" value="/demo/imu"/>
     <joint name="imu_joint" type="fixed">
-        <parent link="chassi"/>
+        <parent link="chassiB"/>
         <child link="imu_frame"/>
         <origin xyz="${imu_x} ${imu_y} ${imu_z}" rpy="0 0 0"/>

File: Computacional/robot/ros_ws/src/autonomous_drive/description/lidar.xacro (robot description, xacro)
@@ -1,10 +1,11 @@
 <?xml version="1.0"?>
 <robot xmlns:xacro="http://www.ros.org/wiki/xacro">
-    <!-- Embora seja dito como um lazer, esse seria a camera, que para a simulação é tratada como um lidar-->
+    <!-- Embora seja dito como um laser, esse seria a câmera, que para a simulação é tratada como um lidar -->
+    <!-- Ou seja, a simulação não está emulando a câmera em si em um LiDAR, mas sim, o seu comportamento, que publicaria em /map  -->
     <xacro:property name="lazer_x" value="0.125"/>
     <xacro:property name="lazer_y" value="0.0"/>
-    <xacro:property name="lazer_z" value="0.15"/>
+    <xacro:property name="lazer_z" value="0.1105"/>
     <joint name="lazer_joint" type="fixed">
-        <parent link="chassi"/>
+        <parent link="chassiA"/>
         <child link="lazer_frame"/>
         <origin xyz="${lazer_x} ${lazer_y} ${lazer_z}" rpy="0.0 0.0 0.0"/>

File: Computacional/robot/ros_ws/src/autonomous_drive/description/marmitron_base.urdf.xacro (robot description, xacro)
@@ -5,3 +5,10 @@
     <xacro:include filename="imu.xacro"/>
     <xacro:include filename="gps.xacro"/>
+    <xacro:include filename="ultrasound.xacro"/>
+    <xacro:ultrasound_sensor name="ultrasound_frente"   parent="chassi" xyz="0.45 0.0 0.075"    rpy="0 0 0"/>
+    <xacro:ultrasound_sensor name="ultrasound_tras"     parent="chassi" xyz="-0.15 0.0 0.075"   rpy="0 0 ${pi}"/>
+    <xacro:ultrasound_sensor name="ultrasound_esquerda" parent="chassi" xyz="0.15 0.175 0.075"  rpy="0 0 ${pi/2}"/>
+    <xacro:ultrasound_sensor name="ultrasound_direita"  parent="chassi" xyz="0.15 -0.175 0.075" rpy="0 0 ${-pi/2}"/>
+    <xacro:ultrasound_sensor name="ultrasound_fe"       parent="chassi" xyz="0.45 0.175 0.075"  rpy="0 0 ${pi/4}"/>
+    <xacro:ultrasound_sensor name="ultrasound_fd"       parent="chassi" xyz="0.45 -0.175 0.075" rpy="0 0 ${-pi/4}"/>
 </robot>

File: Computacional/robot/ros_ws/src/autonomous_drive/description/marmitron_base_sim.urdf.xacro (robot description, xacro)
@@ -6,12 +6,10 @@
     <xacro:include filename="gps.xacro"/>
     <xacro:include filename="robot_controller.xacro"/> <!-- O local com as configurações para simulação -->
-    <xacro:include filename="ultrasound.xacro"/>
-    <xacro:ultrasound_sensor name="ultrasound_frente"   parent="chassi" xyz="0.45 0.0 0.075"    rpy="0 0 0"          topic="ultrasound/front"/>
-    <xacro:ultrasound_sensor name="ultrasound_tras"     parent="chassi" xyz="-0.15 0.0 0.075"   rpy="0 0 ${pi}"      topic="ultrasound/rear"/>
-    <xacro:ultrasound_sensor name="ultrasound_esquerda" parent="chassi" xyz="0.15 0.175 0.075"  rpy="0 0 ${pi/2}"    topic="ultrasound/left"/>
-    <xacro:ultrasound_sensor name="ultrasound_direita"  parent="chassi" xyz="0.15 -0.175 0.075" rpy="0 0 ${-pi/2}"   topic="ultrasound/right"/>
-    <xacro:ultrasound_sensor name="ultrasound_fe"       parent="chassi" xyz="0.45 0.175 0.075"  rpy="0 0 ${pi/4}"    topic="ultrasound/fe"/>
-    <xacro:ultrasound_sensor name="ultrasound_fd"       parent="chassi" xyz="0.45 -0.175 0.075" rpy="0 0 ${-pi/4}"   topic="ultrasound/fd"/>
-    <xacro:ultrasound_sensor name="ultrasound_te"       parent="chassi" xyz="-0.15 0.175 0.075" rpy="0 0 ${3*pi/4}"  topic="ultrasound/te"/>
-    <xacro:ultrasound_sensor name="ultrasound_td"       parent="chassi" xyz="-0.15 -0.175 0.075" rpy="0 0 ${-3*pi/4}" topic="ultrasound/td"/>
+    <xacro:include filename="ultrasound_sim.xacro"/>
+    <xacro:ultrasound_sensor name="ultrasound_frente"   parent="chassiA" xyz="0.2578 0.0 0.0865"    rpy="0 0 0"          topic="ultrasound/front"/>
+    <xacro:ultrasound_sensor name="ultrasound_tras"     parent="chassiA" xyz="-0.2578 0.0 0.0865"   rpy="0 0 ${pi}"      topic="ultrasound/rear"/>
+    <xacro:ultrasound_sensor name="ultrasound_esquerda" parent="chassiA" xyz="0.0 0.175 0.0865"  rpy="0 0 ${pi/2}"    topic="ultrasound/left"/>
+    <xacro:ultrasound_sensor name="ultrasound_direita"  parent="chassiA" xyz="0.0 -0.175 0.0865" rpy="0 0 ${-pi/2}"   topic="ultrasound/right"/>
+    <xacro:ultrasound_sensor name="ultrasound_fe"       parent="chassiA" xyz="0.2578 0.175 0.0865"  rpy="0 0 ${pi/4}"    topic="ultrasound/fe"/>
+    <xacro:ultrasound_sensor name="ultrasound_fd"       parent="chassiA" xyz="0.2578 -0.175 0.0865" rpy="0 0 ${-pi/4}"   topic="ultrasound/fd"/>
 </robot>

File: Computacional/robot/ros_ws/src/autonomous_drive/description/robot_controller.xacro (robot description, xacro)
@@ -9,5 +9,5 @@
     <xacro:property name="lazer_min_angle" value="-0.785"/> <!-- -0.785-->
     <xacro:property name="lazer_max_angle" value="0.785"/>
-    <xacro:property name="lazer_min_range" value="0.5"/>
+    <xacro:property name="lazer_min_range" value="0.3"/>
     <xacro:property name="lazer_max_range" value="12"/>
     <xacro:property name="lazer_topic" value="lidar"/>

File: Computacional/robot/ros_ws/src/autonomous_drive/description/robot_design.xacro (robot description, xacro)
@@ -1,4 +1,4 @@
 <?xml version="1.0"?>
-<!-- Corpo base do robo, suas juntas e localização de sensores -->
+<!-- Corpo base do robô, suas juntas e localização de sensores -->
 <!-- Dimensões são em metros -->
 <robot xmlns:xacro="http://www.ros.org/wiki/xacro">
@@ -6,53 +6,88 @@
     <xacro:include filename="inertials.xacro"/>
     <!-- Chassi -->
-    <xacro:property name="chassi_x" value="0.6"/>
-    <xacro:property name="chassi_y" value="0.35"/>
-    <xacro:property name="chassi_z" value="0.1"/>
-    <xacro:property name="chassi_massa" value="5.3"/>
-    <xacro:property name="chassi_origem" value="0.15 0.0 0.075"/>
-    <xacro:property name="chassi_joint_xyz" value="-0.1 0 0"/>
-    <!-- Rodas trazeiras -->
-    <xacro:property name="roda_raio" value="0.05"/>
+    <xacro:property name="chassiB_x" value="0.507"/>
+    <xacro:property name="chassiB_y" value="0.351"/>
+    <xacro:property name="chassiB_z" value="0.104"/>    <!-- 0.1 (Parte A) + 0.15 (Parte B) -->
+    <xacro:property name="chassiA_x" value="0.516"/>
+    <xacro:property name="chassiA_y" value="0.366"/>
+    <xacro:property name="chassiA_z" value="0.173"/>
+    <!-- Massa do Chassi => (Estimativa Inicial) - 2*(RodasTraseira + RodasApoio) = 6 - 2*(0.055 + 0.05) = 5.79 kg, approx. 5.8 kg -->
+    <xacro:property name="chassiB_massa" value="2"/>
+    <xacro:property name="chassiA_massa" value="3.8"/>
+    <xacro:property name="chassiB_origem" value="0 0 0"/> <!-- "0.254 0.0 0.052" -->
+    <xacro:property name="chassiB_joint_xyz" value="0 0 0.097"/> <!-- 0.045 + 0.052 -->
+    <xacro:property name="chassiA_origem" value="0 0 0"/> <!-- "0.258 0.0 0.087" -->
+    <xacro:property name="chassiA_joint_xyz" value="0 0 0.1185"/> <!-- 0.052 + 0.0865 - 0.02 -->
+    <!-- Rodas dianteiras -->
+    <xacro:property name="roda_raio" value="0.04"/>
     <xacro:property name="roda_comprimento" value="0.04"/>
     <xacro:property name="roda_massa" value="0.5"/>
     <xacro:property name="roda_y" value="0.215"/>
+    <xacro:property name="roda_x" value="0.22"/>
+    <xacro:property name="roda_z" value="-0.052"/>
     <xacro:property name="roda_mu1" value="0.65"/>
     <xacro:property name="roda_mu2" value="0.65"/>
-    <!-- Roda(as) de apio -->
-    <xacro:property name="apoio_raio" value="0.05"/>
-    <xacro:property name="apoio_massa" value="0.5"/>
-    <xacro:property name="apoio_x" value="0.24"/>
+    <!-- Roda(s) de apoio -->
+    <xacro:property name="apoio_raio" value="0.04"/>
+    <xacro:property name="apoio_massa" value="0.35"/>
+    <xacro:property name="apoio_x" value="-0.2"/>
+    <xacro:property name="apoio_y" value="0.125"/>
+    <xacro:property name="apoio_z" value="-0.052"/>
     <xacro:property name="apoio_mu1" value="0.2"/>
     <xacro:property name="apoio_mu2" value="0.2"/>
     <link name="base_link"/>
-    <!-- Chassi -->
-    <joint name="junta_chassi" type="fixed">
+    <!-- Chassi B -->
+    <joint name="junta_chassiB" type="fixed">
         <parent link="base_link"/>
-        <child link="chassi"/>
-        <origin xyz="${chassi_joint_xyz}" rpy="0 0 0"/>
+        <child link="chassiB"/>
+        <origin xyz="${chassiB_joint_xyz}" rpy="0 0 0"/>
     </joint>
-    <link name="chassi">
+    <link name="chassiB">
         <visual>
-            <origin xyz="${chassi_origem}"/>
+            <origin xyz="${chassiB_origem}"/>
             <geometry>
-                <box size="${chassi_x} ${chassi_y} ${chassi_z}"/>
+                <box size="${chassiB_x} ${chassiB_y} ${chassiB_z}"/>
             </geometry>
             <material name="gray"/>
         </visual>
         <collision>
-            <origin xyz="${chassi_origem}"/>
+            <origin xyz="${chassiB_origem}"/>
             <geometry>
-                <box size="${chassi_x} ${chassi_y} ${chassi_z}"/>
+                <box size="${chassiB_x} ${chassiB_y} ${chassiB_z}"/>
             </geometry>
         </collision>
-        <xacro:inertial_box mass="${chassi_massa}" x="${chassi_x}" y="${chassi_y}" z="${chassi_z}">
-            <origin xyz="${chassi_origem}" rpy="0 0 0"/>
+        <xacro:inertial_box mass="${chassiB_massa}" x="${chassiB_x}" y="${chassiB_y}" z="${chassiB_z}">
+            <origin xyz="${chassiB_origem}" rpy="0 0 0"/>
         </xacro:inertial_box>
     </link>
-    <!-- Roda Esquerda Traseira -->
+    <!-- Chassi A -->
+    <joint name="junta_chassiA" type="fixed">
+        <parent link="chassiB"/>
+        <child link="chassiA"/>
+        <origin xyz="${chassiA_joint_xyz}" rpy="0 0 0"/>
+    </joint>
+    <link name="chassiA">
+        <visual>
+            <origin xyz="${chassiA_origem}"/>
+            <geometry>
+                <box size="${chassiA_x} ${chassiA_y} ${chassiA_z}"/>
+            </geometry>
+            <material name="gray"/>
+        </visual>
+        <collision>
+            <origin xyz="${chassiA_origem}"/>
+            <geometry>
+                <box size="${chassiA_x} ${chassiA_y} ${chassiA_z}"/>
+            </geometry>
+        </collision>
+        <xacro:inertial_box mass="${chassiA_massa}" x="${chassiA_x}" y="${chassiA_y}" z="${chassiA_z}">
+            <origin xyz="${chassiA_origem}" rpy="0 0 0"/>
+        </xacro:inertial_box>
+    </link>
+    <!-- Roda Esquerda Dianteira -->
     <joint name="roda_esquerda_joint" type="continuous">
-        <parent link="chassi"/>
+        <parent link="chassiB"/>
         <child link="roda_esquerda"/>
-        <origin xyz="0 ${roda_y} 0" rpy="0 0 0"/>
+        <origin xyz="${roda_x} ${roda_y} ${roda_z}" rpy="0 0 0"/>
         <axis xyz="0 1 0"/>
     </joint>
@@ -75,9 +110,9 @@
         <mu2>${roda_mu2}</mu2>
     </gazebo>
-    <!-- Roda Direita Traseira -->
+    <!-- Roda Direita Dianteira -->
     <joint name="roda_direita_joint" type="continuous">
-        <parent link="chassi"/>
+        <parent link="chassiB"/>
         <child link="roda_direita"/>
-        <origin xyz="0 -${roda_y} 0" rpy="0 0 0"/>
+        <origin xyz="${roda_x} -${roda_y} ${roda_z}" rpy="0 0 0"/>
         <axis xyz="0 1 0"/>
     </joint>
@@ -101,10 +136,11 @@
     </gazebo>
     <!-- Rodas de Apoio -->
-    <joint name="roda_frente_joint" type="fixed">
-        <parent link="chassi"/>
-        <child link="roda_frente"/>
-        <origin xyz="${apoio_x} 0 0"/>
+    <!-- Roda Esquerda -->
+    <joint name="roda_boba1_joint" type="fixed">
+        <parent link="chassiB"/>
+        <child link="roda_boba1"/>
+        <origin xyz="${apoio_x} ${apoio_y} ${apoio_z}"/>
     </joint>
-    <link name="roda_frente">
+    <link name="roda_boba1">
         <visual>
             <geometry>
@@ -122,5 +158,32 @@
         </xacro:inertial_sphere>
     </link>
-    <gazebo reference="roda_frente">
+    <!-- Roda Direita -->
+    <joint name="roda_boba2_joint" type="fixed">
+        <parent link="chassiB"/>
+        <child link="roda_boba2"/>
+        <origin xyz="${apoio_x} -${apoio_y} ${apoio_z}"/>
+    </joint>
+    <link name="roda_boba2">
+        <visual>
+            <geometry>
+                <sphere radius="${apoio_raio}"/>
+            </geometry>
+            <material name="black"/>
+        </visual>
+        <collision>
+            <geometry>
+                <sphere radius="${apoio_raio}"/>
+            </geometry>
+        </collision>
+        <xacro:inertial_sphere mass="${apoio_massa}" radius="${apoio_raio}">
+            <origin xyz="0 0 0" rpy="0 0 0"/>
+        </xacro:inertial_sphere>
+    </link>
+    <gazebo reference="roda_boba1">
+        <self_collide>false</self_collide>
+        <mu1>${apoio_mu1}</mu1>
+        <mu2>${apoio_mu2}</mu2>
+    </gazebo>
+    <gazebo reference="roda_boba2">
         <self_collide>false</self_collide>
         <mu1>${apoio_mu1}</mu1>

File: Computacional/robot/ros_ws/src/autonomous_drive/description/ultrasound.xacro (robot description, xacro)
@@ -16,36 +16,4 @@
             <origin xyz="${xyz}" rpy="${rpy}"/>
         </joint>
-        <gazebo reference="${name}_link">
-            <sensor type="ray" name="${name}_sensor">
-                <pose>0 0 0 0 0 0</pose>
-                <always_on>true</always_on>
-                <update_rate>2</update_rate>
-                <visualize>true</visualize>
-                <ray>
-                    <scan>
-                        <horizontal>
-                            <samples>3</samples>
-                            <resolution>1</resolution>
-                            <min_angle>-0.05</min_angle>
-                            <max_angle>0.05</max_angle>
-                        </horizontal>
-                    </scan>
-                    <range>
-                        <min>0.05</min>
-                        <max>2.0</max>
-                        <resolution>0.01</resolution>
-                    </range>
-                </ray>
-                <plugin name="gazebo_ros_range_${name}" filename="libgazebo_ros_ray_sensor.so">
-                    <ros>
-                        <namespace>/sensor</namespace>
-                        <remapping>~/out:=/${topic}</remapping>
-                    </ros>
-                    <output_type>sensor_msgs/Range</output_type>
-                    <radiation_type>ultrasound</radiation_type>
-                    <frame_name>${name}_link</frame_name>
-                </plugin>
-            </sensor>
-        </gazebo>
     </xacro:macro>
 </robot>
